File: kicad files/alarm.kicad_pcb (KiCad board)
At the start: 2 copper layers, 99 x 80 mm, 18 parts, among them J1 Conn_01x08_Pin, SW1 SW_Push, SW2 SW_Push, SW3 SW_Push, SW5 SW_Push, SW6 SW_Push, SW7 SW_Push, U1 WEMOS_C3_mini

Commit message: Add files via upload
Parts:
- BZ1: footprint Capacitor_THT:CP_Axial_L10.0mm_D4.5mm_P15.00mm_Horizontal -> Buzzer_Beeper:Buzzer_12x9.5RM7.6
- J1: footprint Connector_PinHeader_2.00mm:PinHeader_1x08_P2.00mm_Vertical -> Connector_PinHeader_2.54mm:PinHeader_1x08_P2.54mm_Vertical
- moved BZ1 4.34 mm to (135.0, 36.8)
- moved J1 2.47 mm to (90.6, 73.0)
Routing:
- net +5V: track 91.3 -> 84.7 mm
- net /buzz: track 80.0 -> 85.9 mm, vias 0 -> 1
- net GND: track 122.0 -> 126.3 mm, vias 3 -> 4
- net /BL: track 33.1 -> 36.7 mm
- net /RST: track 34.1 -> 36.7 mm, vias 2 -> 3
- net /SDA: track 7.90 -> 9.89 mm
- net /VCC: track 93.6 -> 91.9 mm, vias 4 -> 5
- net /DC: track 8.34 -> 9.89 mm
- net /CS: track 15.3 -> 13.9 mm
Other:
- board size 99 x 80 mm -> 111.8 x 80 mm
