File: kicad files/alarm.kicad_sch (KiCad schematic)
At the start: 18 parts, among them J1 Conn_01x08_Pin, SW1 SW_Push, SW2 SW_Push, SW3 SW_Push, SW5 SW_Push, SW6 SW_Push, SW7 SW_Push, U1 WEMOS_C3_mini

Commit message: Add files via upload
Parts:
- BZ1: footprint Capacitor_THT:CP_Axial_L10.0mm_D4.5mm_P15.00mm_Horizontal -> Buzzer_Beeper:Buzzer_12x9.5RM7.6
- J1: footprint Connector_PinHeader_2.00mm:PinHeader_1x08_P2.00mm_Vertical -> Connector_PinHeader_2.54mm:PinHeader_1x08_P2.54mm_Vertical
Connections:
- no-connect marks 0 -> 1
Other:
- moved on the sheet: C1
